File: Projects/Client Name/Project Name/Design/rev01/rev01_1/ESC_Project/ESC_Project.kicad_sch (KiCad schematic)
At the start: 0 parts

Commit message: ESC Project skeleton view added by drawing sheets and block diagram
Sheets added and block view drawn
Other:
- added sheet Block Diagram (Block Diagram.kicad_sch)
- added sheet CAN (CAN.kicad_sch)
- added sheet FILTERS (FILTERS.kicad_sch)
- added sheet MCU (MCU.kicad_sch)
- added sheet MOSFET DRIVER (MOSFET DRIVER.kicad_sch)
- added sheet MOSFETs (MOSFETs.kicad_sch)
- added sheet Overview (Overview.kicad_sch)
- note added: "${TITLE}"
- title: Example Project -> ESC Project
